File: sch/VCA.sch (KiCad schematic (older format))
At the start: 0 parts

Commit message: Implementados osciladores de tom (de referência e variável) e volume, circuito ressonante de volume e amplificador controlado por tensão (VCA)
Parts:
- added C1, C3, C5: 4.7pF, symbol C
- added C2: 227pF, symbol C
- added C4, C7: 100nF, symbol C
- added C6: 1nF, symbol C
- added C8: 10uF, symbol CP1
- added CT1: 60pF, symbol CTRIM
- added D1: D_ALT, symbol D_ALT
- added L1: 330uH, symbol L
- added Q1: BC547, TO_SOT_Packages_THT:TO-92_Molded_Narrow, symbol BC547
- added Q1, Q2: 2N5486, symbol Q_NJFET_GSD
- added R1: 10k, symbol R
- added R2: 470k, symbol R
- added R3: 1M, symbol R
- added R4, R5: 4M7, symbol R
- added R6: 1k, symbol R
Connections:
- new net: C1.2, C2.1, C3.1, CT1.1, L1.1
- new net: C3.2, D1.1 (K), Q1.2 (B)
- new net: C4.1, Q1.1 (C), R1.2, R2.1
- new net: C7.1, C8.1, Q1.3 (D), Q2.3 (D), R1.1, R4.1, R6.2
- new net: Q1.1 (G), R2.2
- new net: C6.1, Q1.2 (S), R3.1
- new net: C5.1, R3.2
- new net: C6.2, Q2.1 (G), R4.2, R5.1
- new net +12V: R6.1
- new net AudioIn: C5.2
- new net AudioOut: Q2.2 (S)
- new net GNDREF: C2.2, C4.2, C7.2, C8.2, CT1.2, D1.2 (A), L1.2, Q1.3 (E), R5.2
- new net VolIn: C1.1
