File: sch/mixer.sch (KiCad schematic (older format))
At the start: 11 parts, among them Q1 BC547

Commit message: Implementados osciladores de tom (de referência e variável) e volume, circuito ressonante de volume e amplificador controlado por tensão (VCA)
Parts:
- Q1: TODO (none) -> Buscar um BJT NPN com características de ruído melhores
Changed lines of the file:
@@
 $Descr A4 11693 8268
 encoding utf-8
-Sheet 2 6
+Sheet 2 7
 Title "Theremin2k18"
 Date "2018-09-23"
@@
 F 2 "TO_SOT_Packages_THT:TO-92_Molded_Narrow" H 5450 4125 50  0001 L CIN
 F 3 "" H 5250 4200 50  0001 L CNN
+F 4 "Buscar um BJT NPN com características de ruído melhores" H 5250 4200 60  0001 C CNN "TODO"
 	1    5250 4200
 	1    0    0    -1
