File: sch/pitchVar.sch (KiCad schematic (older format))
At the start: 0 parts

Commit message: Implementados osciladores de tom (de referência e variável) e volume, circuito ressonante de volume e amplificador controlado por tensão (VCA)
Parts:
- added C1: 100nF, symbol C
- added C2: 680pF, symbol C
- added C3, C5: 33nF, symbol C
- added C4: 200pF, symbol C
- added CT1: 60pF, symbol CTRIM
- added L1: 1mH, symbol L
- added Q1: BC547, TO_SOT_Packages_THT:TO-92_Molded_Narrow, symbol BC547
- added R1: 150k, symbol R
- added R2: 33k, symbol R
- added R3, R5: 1k, symbol R
- added R4: 330k, symbol R
Connections:
- new net: C4.1, C5.1, CT1.1, L1.1, R1.1, R5.2
- new net: C1.1, Q1.2 (B), R1.2, R2.1
- new net: C2.2, C3.1, Q1.3 (E), R3.1
- new net +12V: R5.1
- new net Antena: C2.1, C4.2, CT1.2, L1.2, Q1.1 (C), R4.1
- new net GNDREF: C1.2, C3.2, C5.2, R2.2, R3.2
- new net PitchVarOut: R4.2
